File: breakoutsch.sch (EAGLE design)
At the start: 6 parts

Commit message: update to pmod pinout as per http://www.digilentinc.com/Pmods/Digilent-Pmod_%20Interface_Specification.pdf
Parts:
- JP1: device nonolith:HEADER-1X5ROUND -> nonolith:HEADER-1X6ROUND
Connections:
- new net SI: JP1.5
- net 3V3: now also JP1.1; no longer JP1.5
- net CS: now also JP1.6; no longer JP1.2
- net GND: now also JP1.2; no longer JP1.1
- net SCK: now also JP1.3; no longer JP1.4
- net SO: now also JP1.4; no longer JP1.3
Changed lines of the file:
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@@
 <part name="C2" library="nonolith" deviceset="CAP_CERAMIC" device="0603" value="1uF"/>
 <part name="C3" library="nonolith" deviceset="CAP_CERAMIC" device="0603" value="10nF"/>
-<part name="JP1" library="nonolith" deviceset="HEADER-1X5" device="ROUND"/>
+<part name="JP1" library="nonolith" deviceset="HEADER-1X6" device="ROUND"/>
 </parts>
 <sheets>
@@
 <instance part="C2" gate="G$1" x="46.99" y="49.53"/>
 <instance part="C3" gate="G$1" x="63.5" y="74.93"/>
-<instance part="JP1" gate="A" x="-8.89" y="76.2" rot="R180"/>
+<instance part="JP1" gate="A" x="-7.62" y="76.2" rot="R180"/>
 </instances>
 <busses>
@@
 </segment>
 <segment>
-<pinref part="JP1" gate="A" pin="5"/>
-<wire x1="-6.35" y1="81.28" x2="0" y2="81.28" width="0" layer="91"/>
-<label x="1.27" y="81.28" size="1.778" layer="95"/>
+<pinref part="JP1" gate="A" pin="1"/>
+<wire x1="-5.08" y1="68.58" x2="1.27" y2="68.58" width="0" layer="91"/>
+<label x="2.54" y="68.58" size="1.778" layer="95"/>
 </segment>
 </net>
@@
 </segment>
 <segment>
-<wire x1="-6.35" y1="71.12" x2="1.27" y2="71.12" width="0" layer="91"/>
 <label x="1.27" y="71.12" size="1.778" layer="95"/>
-<pinref part="JP1" gate="A" pin="1"/>
+<pinref part="JP1" gate="A" pin="2"/>
+<wire x1="-5.08" y1="71.12" x2="1.27" y2="71.12" width="0" layer="91"/>
 </segment>
 <segment>
@@
 </segment>
 <segment>
-<pinref part="JP1" gate="A" pin="4"/>
-<wire x1="-6.35" y1="78.74" x2="1.27" y2="78.74" width="0" layer="91"/>
-<label x="1.27" y="78.74" size="1.778" layer="95"/>
+<label x="1.27" y="73.66" size="1.778" layer="95"/>
+<pinref part="JP1" gate="A" pin="3"/>
+<wire x1="-5.08" y1="73.66" x2="1.27" y2="73.66" width="0" layer="91"/>
 </segment>
 </net>
@@
 </segment>
 <segment>
-<pinref part="JP1" gate="A" pin="2"/>
-<wire x1="-6.35" y1="73.66" x2="1.27" y2="73.66" width="0" layer="91"/>
-<label x="1.27" y="73.66" size="1.778" layer="95"/>
+<label x="1.27" y="81.28" size="1.778" layer="95"/>
+<pinref part="JP1" gate="A" pin="6"/>
+<wire x1="-5.08" y1="81.28" x2="0" y2="81.28" width="0" layer="91"/>
 </segment>
 </net>
@@
 </segment>
 <segment>
-<pinref part="JP1" gate="A" pin="3"/>
-<wire x1="-6.35" y1="76.2" x2="0" y2="76.2" width="0" layer="91"/>
 <label x="1.27" y="76.2" size="1.778" layer="95"/>
+<pinref part="JP1" gate="A" pin="4"/>
+<wire x1="-5.08" y1="76.2" x2="0" y2="76.2" width="0" layer="91"/>
 </segment>
 </net>
+<net name="SI" class="0">
+<segment>
+<label x="1.27" y="78.74" size="1.778" layer="95"/>
+<pinref part="JP1" gate="A" pin="5"/>
+<wire x1="-5.08" y1="78.74" x2="1.27" y2="78.74" width="0" layer="91"/>
+</segment>
+</net>
